Commit message: Version1.0 completed, but sign of pbvs is differ from paper

File: qfy_dynamixel_description/final_backup19/xacro/final_backup19.xacro (robot description, xacro)
@@ -3,8 +3,9 @@
   <!-- origin of joint connecting battery and mav -->
   <xacro:property name="manipulator_base_joint">
-    <origin xyz="-0.015 0.078 -0.49" rpy="0 0 -0.7853981633974483" />
+    <origin xyz="0 0 -0.03" rpy="1.57 0 0.785398" />
   </xacro:property>
   <xacro:macro name="final_backup19"  params="parent_link">
   <xacro:include filename="$(find qfy_dynamixel_description)/final_backup19/urdf/final_backup19.gazebo" />
+   <!-- add a camera to the manipulator -->
   <link
     name="manipulator_base_link">
@@ -14,5 +15,5 @@
         rpy="0 0 0" />
       <mass
-        value="1.11" />
+        value="0.11" />
       <inertia
         ixx="0.000415"
@@ -54,5 +55,5 @@
         rpy="0 0 0" />
       <mass
-        value="0.126" />
+        value="0.016" />
       <inertia
         ixx="1.696071E-05"
@@ -86,6 +87,6 @@
     type="fixed">
     <origin
-      xyz="-0.045816 -0.0446 0.39074"
-      rpy="0 0 0" />
+      xyz="0 -0.1095 0.113781469737573"
+      rpy="-1.5707963267949 0 3.14159265358979" />
     <parent
       link="manipulator_base_link" />
@@ -102,5 +103,5 @@
         rpy="0 0 0" />
       <mass
-        value="0.153" />
+        value="0.013" />
       <inertia
         ixx="0.02"
@@ -134,6 +135,6 @@
     type="continuous">
     <origin
-      xyz="0 0 -0.07854"
-      rpy="2.1994E-13 1.6974E-16 -3.1416" />
+      xyz="0 0 0.0475000000000002"
+      rpy="-3.1415926 0 -1.57079632678592" />
     <parent
       link="link64" />
@@ -182,6 +183,6 @@
     type="continuous">
     <origin
-      xyz="-0.007 -0.00014931 -0.00018973"
-      rpy="1.5708 -3.7204E-17 9.3147E-50" />
+      xyz="-0.00699999999999945 0 0"
+      rpy="1.5707963267949 0 0" />
     <parent
       link="link106" />
@@ -189,5 +190,5 @@
       link="linkarm" />
     <axis
-      xyz="0 0 1" />
+      xyz="0 0 -1" />
     <dynamics damping="0.2"/>
   </joint>
@@ -199,5 +200,5 @@
         rpy="0 0 0" />
       <mass
-        value="0.06" />
+        value="0.01" />
       <inertia
         ixx="0.002"
@@ -231,6 +232,6 @@
     type="continuous">
     <origin
-      xyz="-0.267847491938725 -0.0315200749343077 -0.000548111211937652"
-      rpy="0 0 0" />
+      xyz="-0.2695 0 0"
+      rpy="0 0 3.1415926" />
     <parent
       link="linkarm" />
@@ -238,5 +239,5 @@
       link="link4" />
     <axis
-      xyz="0 0 1" />
+      xyz="0 0 -1" />
     <dynamics damping="0.2"/>
   </joint>
@@ -248,5 +249,5 @@
         rpy="0 0 0" />
       <mass
-        value="0.06" />
+        value="0.01" />
       <inertia
         ixx="0.01"
@@ -280,6 +281,6 @@
     type="continuous">
     <origin
-      xyz="0.0406502145919447 -0.00888469707381007 -0.00087119563541993"
-      rpy="0 1.57 0" />
+      xyz="0 0 0"
+      rpy="1.5708 0 -3.1416" />
     <parent
       link="link4" />
@@ -287,5 +288,5 @@
       link="link5" />
     <axis
-      xyz="0 0 1" />
+      xyz="0 0 -1" />
     <dynamics damping="0.2"/>
   </joint>
@@ -297,5 +298,5 @@
         rpy="0 0 0" />
       <mass
-        value="0.06" />
+        value="0.02" />
       <inertia
         ixx="0.01"
@@ -334,6 +335,6 @@
     type="continuous">
     <origin
-      xyz="-0.00154477066088465 6.44767978570937E-05 0.0624900000000002"
-      rpy="-1.57079632679487 -1.24154752371065 1.5290817885846" />
+      xyz="0 0 0.10384"
+      rpy="-1.5708 0 0" />
     <parent
       link="link5" />
@@ -341,5 +342,5 @@
       link="link6" />
     <axis
-      xyz="0 0 1" />
+      xyz="0 0 -1" />
     <dynamics damping="0.2"/>
   </joint>
@@ -351,5 +352,5 @@
         rpy="0 0 0" />
       <mass
-        value="0.06" />
+        value="0.03" />
       <inertia
         ixx="0.01"
@@ -388,6 +389,6 @@
     type="continuous">
     <origin
-      xyz="0.0367104165909178 -0.0195888514768517 0.000443884334384581"
-      rpy="1.57079632680098 1.52835246371807 1.19442961140854" />
+      xyz="0 0 0"
+      rpy="1.5708 0 1.5708" />
     <parent
       link="link6" />
@@ -405,5 +406,5 @@
         rpy="0 0 0" />
       <mass
-        value="0.0120765085501768" />
+        value="0.001" />
       <inertia
         ixx="0.01"
@@ -442,6 +443,6 @@
     type="continuous">
     <origin
-      xyz="-0.0144726964004629 0.00108585547271767 0.0399899999999939"
-      rpy="-1.57079632679485 0.289349031429883 -0.1178208167784" />
+      xyz="0 0.0155000000000001 0.0813406770370231"
+      rpy="1.57079632679493 0 -1.5707963267949" />
     <parent
       link="link7" />
@@ -459,5 +460,5 @@
         rpy="0 0 0" />
       <mass
-        value="0.012521326637182" />
+        value="0.001" />
       <inertia
         ixx="0.01"
@@ -496,6 +497,6 @@
     type="continuous">
     <origin
-      xyz="0.0154850896724112 -0.00104013384777768 0.0399900000000045"
-      rpy="-1.57079632679459 0.289349031429808 -0.117820816778367" />
+      xyz="0 -0.0145 0.0813406770370233"
+      rpy="1.57079632679492 0 -1.5707963267949" />
     <parent
       link="link7" />
@@ -503,7 +504,62 @@
       link="finger_left" />
     <axis
-      xyz="0 0 1" />
-    <dynamics damping="0.2"/>
-  </joint>
+      xyz="0 0 -1" />
+    <dynamics damping="0.2"/>
+  </joint>
+<!-- the camera  -->
+ <link
+    name="camera">
+    <inertial>
+      <origin
+        xyz="4.4853E-14 3.6365E-13 -0.005"
+        rpy="0 0 0" />
+      <mass
+        value="0.00676" />
+      <inertia
+        ixx="4.3715E-07"
+        ixy="7.6292E-22"
+        ixz="-2.9141E-18"
+        iyy="4.3715E-07"
+        iyz="-3.0339E-19"
+        izz="7.6163E-07" />
+    </inertial>
+    <visual>
+      <origin
+        xyz="0 0 0"
+        rpy="0 0 0" />
+      <geometry>
+        <mesh
+          filename="package://qfy_dynamixel_description/final_backup19/meshes/camera.stl" />
+      </geometry>
+      <material
+        name="">
+        <color
+          rgba="1 1 1 1" />
+      </material>
+    </visual>
+    <collision>
+      <origin
+        xyz="0 0 0"
+        rpy="0 0 0" />
+      <geometry>
+        <mesh
+          filename="package://qfy_dynamixel_description/final_backup19/meshes/camera.stl" />
+      </geometry>
+    </collision>
+  </link>
+  <joint
+    name="camera_joint"
+    type="fixed">
+    <origin
+      xyz="0.044296 -9.532E-05 0.073724"
+      rpy="-9.0797E-13 8.9782E-12 -1.5708" />
+    <parent
+      link="link7" />
+    <child
+      link="camera" />
+    <axis
+      xyz="0 0 0" />
+  </joint>
+<!-- the plugin of the joint's controller -->
   <transmission name="tran2">
     <type>transmission_interface/SimpleTransmission</type>
